Commit message: Release 4.0
Fix version number to extension version

Add flag to decide whether to parse or ignore joint mimic flag

Handling meshes that inadvertertly duplicate the UV maps

Revert "Handling meshes that inadvertertly duplicate the UV maps"

This reverts commit 23e078403e49f782a3e297527e7c111426d424f0.

Handling meshes that inadvertertly duplicate the UV maps

add prompt checks for path and overwrite for the UI import workflow

fixes articulation root settings

updates version

fixes no joints case

updates expected usd

Add repo codesign so we can publish

change import robot to allow getting articulation root path

Fix issues when Overwriting on import.

Update when saving USD files so it doesn't overload memory or segfaults

code format; remove unecessary includes

add unit test

Inertia Principal Axis; Dynamics damping; Massless Root Link

update default stiffness

Apply 1 suggestion(s) to 1 file(s)

Apply 1 suggestion(s) to 1 file(s)

Apply 1 suggestion(s) to 1 file(s)

Apply 1 suggestion(s) to 1 file(s)

Apply 1 suggestion(s) to 1 file(s)

Apply 1 suggestion(s) to 1 file(s)

Joint Axis is maintained when importing if it's aligned with X, Y or Z parent body axis

Split urdf Parsing and convertion; Add Utility to modify joint drive type

Parse URDF In Memory; Add UI Hooks

Fix ui positioning for the extra frames.

support GLTF meshes in usd

update kit version to 106

Add compatibility to Windows build

adjust for linux+ win build

parse sensors

fix example window UI buttons callbacks

add format options / Code Format

Update Tools; Format code; Update Kit sdk

update repo configs

Update .gitlab-ci.yml file

Update .gitlab-ci.yml file

Fix linux build

disable extension signing

Replace mimic joint from Tendon to Mimic API

Add Articulation to root joint when fixed base

code format

fix symlink message

File: source/extensions/omni.importer.urdf/data/urdf/tests/test_basic.urdf (robot description, URDF)
Before this commit: robot test_basic, 7 links, 6 joints
Links:
- added link finger_link_3, mass 0.7
Joints:
- added joint finger_3_joint: type prismatic, parent palm_link, child finger_link_3, origin xyz=0.30 0 0.05 rpy=0 1.571 0, axis 0 0 1, limit lower=-0.08 upper=0.02 effort=1000.0 velocity=0.5
